File: Version2.0/Version2.0.kicad_pcb (KiCad board)
At the start: 2 copper layers, 83 x 27 mm, 21 parts, among them SW1 SW_Push, U1 DS3231MZ, U2 ESP-12F, U3 TP4056_Module, U4 HT75xx-1-SOT89, U5 DHT11

Commit message: PCB Complete
Routing:
- net GND: vias 0 -> 1
- added copper zone on B.Cu, net GND
- added copper zone on F.Cu, net GND
Other:
- outline, holes or cut-outs redrawn
